File: 555-timer/555-timer.kicad_sch (KiCad schematic)
At the start: 10 parts

Commit message: this work?
Parts:
- gave numbers to parts that had none: 9
Changed lines of the file:
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@@
   (symbol (lib_id "Device:R") (at 37.465 66.04 180) (unit 1)
     (in_bom yes) (on_board yes) (fields_autoplaced)
-    (property "Reference" "R?" (id 0) (at 39.37 64.7699 0)
+    (property "Reference" "R2" (id 0) (at 39.37 64.7699 0)
       (effects (font (size 1.27 1.27)) (justify right))
     )
@@
   (symbol (lib_id "Timer:NE555D") (at 76.835 60.325 0) (unit 1)
     (in_bom yes) (on_board yes) (fields_autoplaced)
-    (property "Reference" "U?" (id 0) (at 78.8544 47.625 0)
-      (effects (font (size 1.27 1.27)) (justify left))
-    )
-    (property "Value" "NE555D" (id 1) (at 78.8544 50.165 0)
+    (property "Reference" "U1" (id 0) (at 78.8544 46.99 0)
+      (effects (font (size 1.27 1.27)) (justify left))
+    )
+    (property "Value" "NE555D" (id 1) (at 78.8544 49.53 0)
       (effects (font (size 1.27 1.27)) (justify left))
     )
@@
   (symbol (lib_id "Device:LED") (at 116.84 34.29 90) (unit 1)
     (in_bom yes) (on_board yes) (fields_autoplaced)
-    (property "Reference" "D?" (id 0) (at 120.65 34.6074 90)
+    (property "Reference" "D1" (id 0) (at 120.65 34.6074 90)
       (effects (font (size 1.27 1.27)) (justify right))
     )
@@
   (symbol (lib_id "Device:R") (at 116.84 46.355 0) (unit 1)
     (in_bom yes) (on_board yes) (fields_autoplaced)
-    (property "Reference" "R?" (id 0) (at 119.38 45.0849 0)
+    (property "Reference" "R3" (id 0) (at 119.38 45.0849 0)
       (effects (font (size 1.27 1.27)) (justify left))
     )
@@
   (symbol (lib_id "Connector:Conn_01x02_Male") (at 73.66 36.195 90) (unit 1)
     (in_bom yes) (on_board yes) (fields_autoplaced)
-    (property "Reference" "J?" (id 0) (at 77.47 35.5599 90)
+    (property "Reference" "J1" (id 0) (at 77.47 35.5599 90)
       (effects (font (size 1.27 1.27)) (justify right))
     )
@@
   (symbol (lib_id "Device:C_Polarized") (at 37.465 83.82 0) (unit 1)
     (in_bom yes) (on_board yes) (fields_autoplaced)
-    (property "Reference" "C?" (id 0) (at 40.64 81.6609 0)
+    (property "Reference" "C1" (id 0) (at 40.64 81.6609 0)
       (effects (font (size 1.27 1.27)) (justify left))
     )
@@
   (symbol (lib_id "Device:R") (at 37.465 46.355 0) (unit 1)
     (in_bom yes) (on_board yes) (fields_autoplaced)
-    (property "Reference" "R?" (id 0) (at 39.37 45.0849 0)
+    (property "Reference" "R1" (id 0) (at 39.37 45.0849 0)
       (effects (font (size 1.27 1.27)) (justify left))
     )
@@
   (symbol (lib_id "Device:C") (at 55.245 74.295 0) (unit 1)
     (in_bom yes) (on_board yes) (fields_autoplaced)
-    (property "Reference" "C?" (id 0) (at 58.42 73.0249 0)
+    (property "Reference" "C2" (id 0) (at 58.42 73.0249 0)
       (effects (font (size 1.27 1.27)) (justify left))
     )
@@
   (symbol (lib_id "Device:LED") (at 116.84 81.915 90) (unit 1)
     (in_bom yes) (on_board yes) (fields_autoplaced)
-    (property "Reference" "D?" (id 0) (at 120.65 82.2324 90)
+    (property "Reference" "D4" (id 0) (at 120.65 82.2324 90)
       (effects (font (size 1.27 1.27)) (justify right))
     )
@@
     )
     (path "/e76ec524-408a-4daa-89f6-0edfdbcfb621"
-      (reference "C?") (unit 1) (value "10µF") (footprint "")
+      (reference "C1") (unit 1) (value "10µF") (footprint "")
     )
     (path "/eb473bfd-fc2d-4cf0-8714-6b7dd95b0a03"
-      (reference "C?") (unit 1) (value "0.01µF") (footprint "")
+      (reference "C2") (unit 1) (value "0.01µF") (footprint "")
     )
     (path "/62a1f3d4-027d-4ecf-a37a-6fcf4263e9d2"
-      (reference "D?") (unit 1) (value "LED") (footprint "")
+      (reference "D1") (unit 1) (value "LED") (footprint "")
     )
     (path "/f4a8afbe-ed68-4253-959f-6be4d2cbf8c5"
-      (reference "D?") (unit 1) (value "LED") (footprint "")
+      (reference "D4") (unit 1) (value "LED") (footprint "")
     )
     (path "/e0c7ddff-8c90-465f-be62-21fb49b059fa"
-      (reference "J?") (unit 1) (value "Conn_01x02_Male") (footprint "")
+      (reference "J1") (unit 1) (value "Conn_01x02_Male") (footprint "")
+    )
+    (path "/ea2ea877-1ce1-4cd6-ad19-1da87f51601d"
+      (reference "R1") (unit 1) (value "1k") (footprint "")
     )
     (path "/02538207-54a8-4266-8d51-23871852b2ff"
-      (reference "R?") (unit 1) (value "10k") (footprint "")
+      (reference "R2") (unit 1) (value "10k") (footprint "")
     )
     (path "/84d4e166-b429-409a-ab37-c6a10fd82ff5"
-      (reference "R?") (unit 1) (value "1k") (footprint "")
+      (reference "R3") (unit 1) (value "1k") (footprint "")
     )
     (path "/89c9afdc-c346-4300-a392-5f9dd8c1e5bd"
       (reference "R?") (unit 1) (value "1k") (footprint "")
     )
-    (path "/ea2ea877-1ce1-4cd6-ad19-1da87f51601d"
-      (reference "R?") (unit 1) (value "1k") (footprint "")
-    )
     (path "/0b9f21ed-3d41-4f23-ae45-74117a5f3153"
-      (reference "U?") (unit 1) (value "NE555D") (footprint "Package_SO:SOIC-8_3.9x4.9mm_P1.27mm")
-    )
-  )
+      (reference "U1") (unit 1) (value "NE555D") (footprint "Package_SO:SOIC-8_3.9x4.9mm_P1.27mm")
+    )
+  )

Commit message: AAAAAAAAAAAAAAAAAAAAAAAAAH
Parts:
- C1: footprint (none) -> Capacitor_Tantalum_SMD:CP_EIA-3216-18_Kemet-A_Pad1.58x1.35mm_HandSolder
- C2: footprint (none) -> Capacitor_SMD:C_0805_2012Metric_Pad1.18x1.45mm_HandSolder
- D1: footprint (none) -> LED_SMD:LED_1206_3216Metric_Pad1.42x1.75mm_HandSolder
- D2: renamed from D4; footprint (none) -> LED_SMD:LED_1206_3216Metric_Pad1.42x1.75mm_HandSolder
- J1: footprint (none) -> Connector_JST:JST_EH_S2B-EH_1x02_P2.50mm_Horizontal
- R1, R2, R3: footprint (none) -> Resistor_SMD:R_0805_2012Metric_Pad1.20x1.40mm_HandSolder
- R4: renamed from R?; footprint (none) -> Resistor_SMD:R_0805_2012Metric_Pad1.20x1.40mm_HandSolder
- U1: footprint Package_SO:SOIC-8_3.9x4.9mm_P1.27mm -> Package_SO:SOIC-8-1EP_3.9x4.9mm_P1.27mm_EP2.29x3mm
Changed lines of the file:
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@@
       (effects (font (size 1.27 1.27)) (justify right))
     )
-    (property "Footprint" "" (id 2) (at 39.243 66.04 90)
+    (property "Footprint" "Resistor_SMD:R_0805_2012Metric_Pad1.20x1.40mm_HandSolder" (id 2) (at 39.243 66.04 90)
       (effects (font (size 1.27 1.27)) hide)
     )
@@
       (effects (font (size 1.27 1.27)) (justify left))
     )
-    (property "Footprint" "Package_SO:SOIC-8_3.9x4.9mm_P1.27mm" (id 2) (at 98.425 70.485 0)
+    (property "Footprint" "Package_SO:SOIC-8-1EP_3.9x4.9mm_P1.27mm_EP2.29x3mm" (id 2) (at 98.425 70.485 0)
       (effects (font (size 1.27 1.27)) hide)
     )
@@
       (effects (font (size 1.27 1.27)) (justify right))
     )
-    (property "Footprint" "" (id 2) (at 116.84 34.29 0)
+    (property "Footprint" "LED_SMD:LED_1206_3216Metric_Pad1.42x1.75mm_HandSolder" (id 2) (at 116.84 34.29 0)
       (effects (font (size 1.27 1.27)) hide)
     )
@@
   (symbol (lib_id "power:GND") (at 73.66 100.965 0) (unit 1)
     (in_bom yes) (on_board yes) (fields_autoplaced)
-    (property "Reference" "#PWR?" (id 0) (at 73.66 107.315 0)
+    (property "Reference" "#PWR0101" (id 0) (at 73.66 107.315 0)
       (effects (font (size 1.27 1.27)) hide)
     )
@@
   (symbol (lib_id "power:+9V") (at 116.84 27.305 0) (unit 1)
     (in_bom yes) (on_board yes) (fields_autoplaced)
-    (property "Reference" "#PWR?" (id 0) (at 116.84 31.115 0)
+    (property "Reference" "#PWR0106" (id 0) (at 116.84 31.115 0)
       (effects (font (size 1.27 1.27)) hide)
     )
@@
   (symbol (lib_id "power:+9V") (at 37.465 39.37 0) (unit 1)
     (in_bom yes) (on_board yes) (fields_autoplaced)
-    (property "Reference" "#PWR?" (id 0) (at 37.465 43.18 0)
+    (property "Reference" "#PWR0102" (id 0) (at 37.465 43.18 0)
       (effects (font (size 1.27 1.27)) hide)
     )
@@
   (symbol (lib_id "power:GND") (at 76.2 28.575 180) (unit 1)
     (in_bom yes) (on_board yes) (fields_autoplaced)
-    (property "Reference" "#PWR?" (id 0) (at 76.2 22.225 0)
+    (property "Reference" "#PWR0105" (id 0) (at 76.2 22.225 0)
       (effects (font (size 1.27 1.27)) hide)
     )
@@
       (effects (font (size 1.27 1.27)) (justify left))
     )
-    (property "Footprint" "" (id 2) (at 115.062 46.355 90)
+    (property "Footprint" "Resistor_SMD:R_0805_2012Metric_Pad1.20x1.40mm_HandSolder" (id 2) (at 115.062 46.355 90)
       (effects (font (size 1.27 1.27)) hide)
     )
@@
   (symbol (lib_id "Device:R") (at 116.84 64.135 0) (unit 1)
     (in_bom yes) (on_board yes) (fields_autoplaced)
-    (property "Reference" "R?" (id 0) (at 119.38 62.8649 0)
+    (property "Reference" "R4" (id 0) (at 119.38 62.8649 0)
       (effects (font (size 1.27 1.27)) (justify left))
     )
@@
       (effects (font (size 1.27 1.27)) (justify left))
     )
-    (property "Footprint" "" (id 2) (at 115.062 64.135 90)
+    (property "Footprint" "Resistor_SMD:R_0805_2012Metric_Pad1.20x1.40mm_HandSolder" (id 2) (at 115.062 64.135 90)
       (effects (font (size 1.27 1.27)) hide)
     )
@@
   )
   (symbol (lib_id "power:+9V") (at 76.835 46.355 0) (unit 1)
-    (in_bom yes) (on_board yes) (fields_autoplaced)
-    (property "Reference" "#PWR?" (id 0) (at 76.835 50.165 0)
-      (effects (font (size 1.27 1.27)) hide)
-    )
-    (property "Value" "+9V" (id 1) (at 76.835 40.64 0))
+    (in_bom yes) (on_board yes)
+    (property "Reference" "#PWR0103" (id 0) (at 76.835 50.165 0)
+      (effects (font (size 1.27 1.27)) hide)
+    )
+    (property "Value" "+9V" (id 1) (at 77.47 41.91 0))
     (property "Footprint" "" (id 2) (at 76.835 46.355 0)
       (effects (font (size 1.27 1.27)) hide)
@@
   (symbol (lib_id "power:+9V") (at 73.66 28.575 0) (unit 1)
     (in_bom yes) (on_board yes) (fields_autoplaced)
-    (property "Reference" "#PWR?" (id 0) (at 73.66 32.385 0)
+    (property "Reference" "#PWR0104" (id 0) (at 73.66 32.385 0)
       (effects (font (size 1.27 1.27)) hide)
     )
@@
       (effects (font (size 1.27 1.27)) (justify right) hide)
     )
-    (property "Footprint" "" (id 2) (at 73.66 36.195 0)
+    (property "Footprint" "Connector_JST:JST_EH_S2B-EH_1x02_P2.50mm_Horizontal" (id 2) (at 73.66 36.195 0)
       (effects (font (size 1.27 1.27)) hide)
     )
@@
       (effects (font (size 1.27 1.27)) (justify left))
     )
-    (property "Footprint" "" (id 2) (at 38.4302 87.63 0)
+    (property "Footprint" "Capacitor_Tantalum_SMD:CP_EIA-3216-18_Kemet-A_Pad1.58x1.35mm_HandSolder" (id 2) (at 38.4302 87.63 0)
       (effects (font (size 1.27 1.27)) hide)
     )
@@
       (effects (font (size 1.27 1.27)) (justify left))
     )
-    (property "Footprint" "" (id 2) (at 35.687 46.355 90)
+    (property "Footprint" "Resistor_SMD:R_0805_2012Metric_Pad1.20x1.40mm_HandSolder" (id 2) (at 35.687 46.355 90)
       (effects (font (size 1.27 1.27)) hide)
     )
@@
       (effects (font (size 1.27 1.27)) (justify left))
     )
-    (property "Footprint" "" (id 2) (at 56.2102 78.105 0)
+    (property "Footprint" "Capacitor_SMD:C_0805_2012Metric_Pad1.18x1.45mm_HandSolder" (id 2) (at 56.2102 78.105 0)
       (effects (font (size 1.27 1.27)) hide)
     )
@@
   (symbol (lib_id "Device:LED") (at 116.84 81.915 90) (unit 1)
     (in_bom yes) (on_board yes) (fields_autoplaced)
-    (property "Reference" "D4" (id 0) (at 120.65 82.2324 90)
+    (property "Reference" "D2" (id 0) (at 120.65 82.2324 90)
       (effects (font (size 1.27 1.27)) (justify right))
     )
@@
       (effects (font (size 1.27 1.27)) (justify right))
     )
-    (property "Footprint" "" (id 2) (at 116.84 81.915 0)
+    (property "Footprint" "LED_SMD:LED_1206_3216Metric_Pad1.42x1.75mm_HandSolder" (id 2) (at 116.84 81.915 0)
       (effects (font (size 1.27 1.27)) hide)
     )
@@
   (symbol_instances
     (path "/6a0919c2-460c-4229-b872-14e318e1ba8b"
-      (reference "#PWR?") (unit 1) (value "GND") (footprint "")
+      (reference "#PWR0101") (unit 1) (value "GND") (footprint "")
+    )
+    (path "/799e761c-1426-40e9-a069-1f4cb353bfaa"
+      (reference "#PWR0102") (unit 1) (value "+9V") (footprint "")
+    )
+    (path "/8cb2cd3a-4ef9-4ae5-b6bc-2b1d16f657d6"
+      (reference "#PWR0103") (unit 1) (value "+9V") (footprint "")
+    )
+    (path "/d66d3c12-11ce-4566-9a45-962e329503d8"
+      (reference "#PWR0104") (unit 1) (value "+9V") (footprint "")
+    )
+    (path "/844d7d7a-b386-45a8-aaf6-bf41bbcb43b5"
+      (reference "#PWR0105") (unit 1) (value "GND") (footprint "")
     )
     (path "/6b91a3ee-fdcd-4bfe-ad57-c8d5ea9903a8"
-      (reference "#PWR?") (unit 1) (value "+9V") (footprint "")
-    )
-    (path "/799e761c-1426-40e9-a069-1f4cb353bfaa"
-      (reference "#PWR?") (unit 1) (value "+9V") (footprint "")
-    )
-    (path "/844d7d7a-b386-45a8-aaf6-bf41bbcb43b5"
-      (reference "#PWR?") (unit 1) (value "GND") (footprint "")
-    )
-    (path "/8cb2cd3a-4ef9-4ae5-b6bc-2b1d16f657d6"
-      (reference "#PWR?") (unit 1) (value "+9V") (footprint "")
-    )
-    (path "/d66d3c12-11ce-4566-9a45-962e329503d8"
-      (reference "#PWR?") (unit 1) (value "+9V") (footprint "")
+      (reference "#PWR0106") (unit 1) (value "+9V") (footprint "")
     )
     (path "/e76ec524-408a-4daa-89f6-0edfdbcfb621"
-      (reference "C1") (unit 1) (value "10µF") (footprint "")
+      (reference "C1") (unit 1) (value "10µF") (footprint "Capacitor_Tantalum_SMD:CP_EIA-3216-18_Kemet-A_Pad1.58x1.35mm_HandSolder")
     )
     (path "/eb473bfd-fc2d-4cf0-8714-6b7dd95b0a03"
-      (reference "C2") (unit 1) (value "0.01µF") (footprint "")
+      (reference "C2") (unit 1) (value "0.01µF") (footprint "Capacitor_SMD:C_0805_2012Metric_Pad1.18x1.45mm_HandSolder")
     )
     (path "/62a1f3d4-027d-4ecf-a37a-6fcf4263e9d2"
-      (reference "D1") (unit 1) (value "LED") (footprint "")
+      (reference "D1") (unit 1) (value "LED") (footprint "LED_SMD:LED_1206_3216Metric_Pad1.42x1.75mm_HandSolder")
     )
     (path "/f4a8afbe-ed68-4253-959f-6be4d2cbf8c5"
-      (reference "D4") (unit 1) (value "LED") (footprint "")
+      (reference "D2") (unit 1) (value "LED") (footprint "LED_SMD:LED_1206_3216Metric_Pad1.42x1.75mm_HandSolder")
     )
     (path "/e0c7ddff-8c90-465f-be62-21fb49b059fa"
-      (reference "J1") (unit 1) (value "Conn_01x02_Male") (footprint "")
+      (reference "J1") (unit 1) (value "Conn_01x02_Male") (footprint "Connector_JST:JST_EH_S2B-EH_1x02_P2.50mm_Horizontal")
     )
     (path "/ea2ea877-1ce1-4cd6-ad19-1da87f51601d"
-      (reference "R1") (unit 1) (value "1k") (footprint "")
+      (reference "R1") (unit 1) (value "1k") (footprint "Resistor_SMD:R_0805_2012Metric_Pad1.20x1.40mm_HandSolder")
     )
     (path "/02538207-54a8-4266-8d51-23871852b2ff"
-      (reference "R2") (unit 1) (value "10k") (footprint "")
+      (reference "R2") (unit 1) (value "10k") (footprint "Resistor_SMD:R_0805_2012Metric_Pad1.20x1.40mm_HandSolder")
     )
     (path "/84d4e166-b429-409a-ab37-c6a10fd82ff5"
-      (reference "R3") (unit 1) (value "1k") (footprint "")
+      (reference "R3") (unit 1) (value "1k") (footprint "Resistor_SMD:R_0805_2012Metric_Pad1.20x1.40mm_HandSolder")
     )
     (path "/89c9afdc-c346-4300-a392-5f9dd8c1e5bd"
-      (reference "R?") (unit 1) (value "1k") (footprint "")
+      (reference "R4") (unit 1) (value "1k") (footprint "Resistor_SMD:R_0805_2012Metric_Pad1.20x1.40mm_HandSolder")
     )
     (path "/0b9f21ed-3d41-4f23-ae45-74117a5f3153"
-      (reference "U1") (unit 1) (value "NE555D") (footprint "Package_SO:SOIC-8_3.9x4.9mm_P1.27mm")
-    )
-  )
+      (reference "U1") (unit 1) (value "NE555D") (footprint "Package_SO:SOIC-8-1EP_3.9x4.9mm_P1.27mm_EP2.29x3mm")
+    )
+  )
